File: hardware/keurig-filler/keurig-filler/keurig-filler.kicad_pcb (KiCad board)
At the start: 2 copper layers, 86.1 x 64.8 mm, 16 parts, among them J1 To Level Sensor in Source, J2 To Level Sensor in Keurig, J3 To Flow Sensor, J4 To Water Pump, J5 Voltage Regulator Board, J6 To Power Adapter Jack, K1 KF0602D, Q1 DMG2305UX-7, U1 Pico

Commit message: Created v2 board design
Adding HC-05 bluetooth module, LCD screen (over I2C) and a FRAM (over SPI).  Full firmware support for the FRAM and LCD not yet added.

Gerbers not yet regenerated.
Parts:
- removed REF** (x4): MountingHole_2.5mm, MountingHole:MountingHole_2.5mm
- removed REF**: OSHW-Logo2_14.6x12mm_SilkScreen, Symbol:OSHW-Logo2_14.6x12mm_SilkScreen
- added J7: To LCD Module, Connector_PinHeader_2.54mm:PinHeader_1x04_P2.54mm_Vertical, F.Cu at (77.7, 80.1)
- added J8: To HC-05 Module, Connector_PinHeader_2.54mm:PinHeader_1x06_P2.54mm_Vertical, F.Cu at (50.4, 24.4)
- added Q2: 2N7002, Package_TO_SOT_SMD:SOT-23, B.Cu at (38.4, 52.1)
- added Q3: 2N7002, Package_TO_SOT_SMD:SOT-23, B.Cu at (34.8, 49.5)
- added Q4: 2N7002, Package_TO_SOT_SMD:SOT-23, B.Cu at (34.5, 64.0)
- added Q5: 2N7002, Package_TO_SOT_SMD:SOT-23, B.Cu at (39.0, 66.8)
- added Q6: 2N7002, Package_TO_SOT_SMD:SOT-23, B.Cu at (37.3, 72.9)
- added R10: 4k7, Resistor_SMD:R_0805_2012Metric_Pad1.20x1.40mm_HandSolder, F.Cu at (60.7, 36.1)
- added R11: 4k7, Resistor_SMD:R_0805_2012Metric_Pad1.20x1.40mm_HandSolder, B.Cu at (39.0, 69.7)
- added R12: 4k7, Resistor_SMD:R_0805_2012Metric_Pad1.20x1.40mm_HandSolder, F.Cu at (44.3, 37.7)
- added R13: 4k7, Resistor_SMD:R_0805_2012Metric_Pad1.20x1.40mm_HandSolder, B.Cu at (37.2, 75.9)
- added R2: 4k7, Resistor_SMD:R_0805_2012Metric_Pad1.20x1.40mm_HandSolder, B.Cu at (41.7, 49.8)
- added R3: 4k7, Resistor_SMD:R_0805_2012Metric_Pad1.20x1.40mm_HandSolder, B.Cu at (37.6, 47.2)
- added R4: 4k7, Resistor_SMD:R_0805_2012Metric_Pad1.20x1.40mm_HandSolder, B.Cu at (38.3, 55.4)
- added R5: 4k7, Resistor_SMD:R_0805_2012Metric_Pad1.20x1.40mm_HandSolder, F.Cu at (34.0, 54.3)
- added R6: 1k, Resistor_SMD:R_0805_2012Metric_Pad1.20x1.40mm_HandSolder, F.Cu at (82.9, 35.1)
- added R7: 1k, Resistor_SMD:R_0805_2012Metric_Pad1.20x1.40mm_HandSolder, F.Cu at (79.6, 30.1)
- added R8: 4k7, Resistor_SMD:R_0805_2012Metric_Pad1.20x1.40mm_HandSolder, F.Cu at (64.0, 41.0)
- added R9: 4k7, Resistor_SMD:R_0805_2012Metric_Pad1.20x1.40mm_HandSolder, B.Cu at (34.5, 66.9)
- added U2: MB85RS64V, SnapEDA Library:SOIC127P600X155-8_R159_68_374R15, F.Cu at (58.7, 74.9)
- Q1: value DMG2305UX-7 -> ‎SSM3J371R,LF‎
Connections:
- U1 pad 1: UART_TX0 -> Net-(U1-Pad1)
- U1 pad 16: Net-(U1-Pad16) -> UART_TX0
- U1 pad 17: Net-(U1-Pad17) -> UART_RX0
- U1 pad 19: Net-(U1-Pad19) -> ~UART_KEY
- U1 pad 2: UART_RX0 -> Net-(U1-Pad2)
- U1 pad 25: MOSI -> MOSI0
- U1 pad 34: GND -> Net-(U1-Pad34)
Routing:
- net +5V: track 7.68 -> 101.8 mm, vias 0 -> 5
- net SDA_5V: track 0.00 -> 71.7 mm, vias 0 -> 3
- net HC05_RX: track 0.00 -> 65.1 mm, vias 0 -> 6
- net SCL_5V: track 0.00 -> 63.3 mm, vias 0 -> 5
- net HC05_TX: track 0.00 -> 61.6 mm, vias 0 -> 4
- net ~HC05_KEY: track 0.00 -> 56.4 mm, vias 0 -> 4
- net +3V3: track 0.00 -> 15.4 mm, vias 0 -> 5
- net MOSI0: track 0.00 -> 15.3 mm, vias 0 -> 1
- net SCK0: track 0.00 -> 13.6 mm
- net MISO0: track 0.00 -> 12.3 mm
- net UART_RX0: track 0.00 -> 9.88 mm
- net SPI_CS0: track 0.00 -> 9.76 mm
- net SCL0: track 0.00 -> 9.21 mm
- net ~UART_KEY: track 0.00 -> 7.82 mm
- net GND: track 2.06 -> 9.68 mm, vias 1 -> 3
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Other:
- board text added: "Keurig Filler v2.0"
- board text removed: "Keurig Filler v1.0"

Commit message: Update gerbers for v2
Parts:
- added REF**: OSHW-Logo2_14.6x12mm_SilkScreen, Symbol:OSHW-Logo2_14.6x12mm_SilkScreen, F.Cu at (69.5, 70.9)
