File: hardware/keurig-filler/keurig-filler/keurig-filler.sch (KiCad schematic (older format))
At the start: 11 parts, among them J1 To Level Sensor in Source, J2 To Level Sensor in Keurig, J3 To Flow Sensor, J4 To Water Pump, J5 Voltage Regulator Board, J6 To Power Adapter Jack, K1 KF0602D, Q1 ‎SSM3J371R,LF‎, U1 Pico

Commit message: Created v2 board design
Adding HC-05 bluetooth module, LCD screen (over I2C) and a FRAM (over SPI).  Full firmware support for the FRAM and LCD not yet added.

Gerbers not yet regenerated.
Parts:
- added J7: To LCD Module, Connector_PinHeader_2.54mm:PinHeader_1x04_P2.54mm_Vertical, symbol Connector:Conn_01x04_Female
- added J8: To HC-05 Module, Connector_PinHeader_2.54mm:PinHeader_1x06_P2.54mm_Vertical, symbol Connector:Conn_01x06_Female
- added Q2, Q3, Q4, Q5, Q6: 2N7002, Package_TO_SOT_SMD:SOT-23, symbol Transistor_FET:2N7002
- added R10, R11, R12, R13, R2, R3, R4, R5, R8, R9: 4k7, Resistor_SMD:R_0805_2012Metric_Pad1.20x1.40mm_HandSolder, symbol Device:R
- added R6, R7: 1k, Resistor_SMD:R_0805_2012Metric_Pad1.20x1.40mm_HandSolder, symbol Device:R
- added U2: MB85RS64V, SnapEDA Library:SOIC127P600X155-8_R159_68_374R15, symbol MB85RS64V:MB85RS64V
Connections:
- net +3V3: now also Q2.1 (G), Q3.1 (G), Q4.1 (G), Q5.1 (G), Q6.1 (G), R11.2, R13.2, R4.2, R5.2, R9.2, U2.3 (~WP), U2.7 (~HOLD), U2.8 (VCC)
- net +5V: now also J7.2 (Pin_2), J8.2 (Pin_2), R10.2, R12.2, R2.2, R3.2, R8.2
- net ADC0: now also R7.1
- net ADC1: now also R6.1
- net GND: now also J7.1 (Pin_1), J8.3 (Pin_3), R6.2, R7.2, U2.4 (GND); no longer U1.34 (GPIO28_ADC2)
- net MISO0: now also U2.2 (MISO)
- net SCK0: now also U2.6 (SCK)
- net SCL0: now also Q2.2 (S), R4.1
- net SDA0: now also Q3.2 (S), R5.1
- net SPI_CS0: now also U2.1 (~CS)
- net UART_RX0: now also U1.17 (GPIO13), Q5.2 (S), R11.1; no longer U1.2 (GPIO1)
- net UART_TX0: now also U1.16 (GPIO12), Q4.2 (S), R9.1; no longer U1.1 (GPIO0)
- net ~UART_KEY: now reaches U1.19 (GPIO14)
- net ~UART_KEY: now also Q6.2 (S), R13.1
- net MOSI renamed MOSI0
- net MOSI0: now also U2.5 (MOSI)
- new net HC05_RX: J8.5 (Pin_5), Q4.3 (D), R8.1
- new net HC05_TX: J8.4 (Pin_4), Q5.3 (D), R10.1
- new net SCL_5V: J7.4 (Pin_4), Q2.3 (D), R2.1
- new net SDA_5V: J7.3 (Pin_3), Q3.3 (D), R3.1
- new net ~HC05_KEY: J8.1 (Pin_1), Q6.3 (D), R12.1
- no-connect marks 17 -> 18

Commit message: Update gerbers for v2
Changed lines of the file:
@@
 NoConn ~ 5310 2590
 NoConn ~ 5310 3290
+$Comp
+L Graphic:Logo_Open_Hardware_Large #LOGO1
+U 1 1 61EDAA38
+P 6350 7170
+F 0 "#LOGO1" H 6350 7670 50  0001 C CNN
+F 1 "Logo_Open_Hardware_Large" H 6350 6770 50  0001 C CNN
+F 2 "" H 6350 7170 50  0001 C CNN
+F 3 "~" H 6350 7170 50  0001 C CNN
+	1    6350 7170
+	1    0    0    -1
+$EndComp
 $EndSCHEMATC
